File: Schematic-and-BOM/MightyWatt R3.brd (EAGLE design)
At the start: 64.8 x 53.3 mm, 93 parts, among them IC1 TLV271IDBVR, IC2 MAX4619EUE, IC3 OPA365AIDBVR, IC4 TS5A3166, IC5 INA225, IC6 ADS1115IDGST, IC7 TLV2372IDGK, IC8 AD5691RAD5691R, IC9 LM2766M6, T1 IXTH75N10L2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

Commit message: Fixed schematic
Parts:
- C1: value DNP -> 2u2/16V
- C2: value 100n -> DNP
- R3: value DNP -> 0R
- R6: value 1k -> 75R
Changed lines of the file:
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@@
 <attribute name="VALUE" x="1.349375" y="20.081875" size="1.27" layer="27" rot="R270"/>
 </element>
-<element name="R6" library="rcl" package="R0603" value="1k" x="10.00125" y="19.764375" smashed="yes" rot="R180">
+<element name="R6" library="rcl" package="R0603" value="75R" x="10.00125" y="19.764375" smashed="yes" rot="R180">
 <attribute name="NAME" x="9.921875" y="19.05" size="0.8128" layer="25" font="vector" rot="R180"/>
 <attribute name="VALUE" x="10.63625" y="21.669375" size="1.27" layer="27" rot="R180"/>
@@
 <attribute name="VALUE" x="2.498725" y="9.445625" size="2.0828" layer="27" ratio="10" rot="SR0"/>
 </element>
-<element name="C2" library="rcl" package="C0603" value="100n" x="14.684375" y="9.36625" smashed="yes">
+<element name="C2" library="rcl" package="C0603" value="DNP" x="14.684375" y="9.36625" smashed="yes">
 <attribute name="NAME" x="16.271875" y="8.969375" size="0.8128" layer="25" font="vector"/>
 <attribute name="VALUE" x="14.049375" y="7.46125" size="1.27" layer="27"/>
 </element>
-<element name="R3" library="rcl" package="R0603" value="DNP" x="14.684375" y="7.858125" smashed="yes" rot="R180">
+<element name="R3" library="rcl" package="R0603" value="0R" x="14.684375" y="7.858125" smashed="yes" rot="R180">
 <attribute name="NAME" x="17.700625" y="8.255" size="0.8128" layer="25" font="vector" rot="R180"/>
 <attribute name="VALUE" x="15.319375" y="9.763125" size="1.27" layer="27" rot="R180"/>
 </element>
-<element name="C1" library="rcl" package="C1206" value="DNP" x="11.509375" y="10.715625" smashed="yes" rot="R270">
+<element name="C1" library="rcl" package="C1206" value="2u2/16V" x="11.509375" y="10.715625" smashed="yes" rot="R270">
 <attribute name="NAME" x="9.2075" y="10.239375" size="0.8128" layer="25" font="vector"/>
 <attribute name="VALUE" x="8.969375" y="11.985625" size="1.27" layer="27" rot="R270"/>

Commit message: Schematic fix
- Proper symbols of bi-directional TVS were added to the schematic.
- Order of switching current and voltage ranges was upgraded to decrease
spikes.
- Guide was updated.
Parts:
- D1: device diode-tvs:SMC -> kaktus:SMC
- D6, D7, D8: device diode:DO-214AC -> kaktus:DO-214AC
Changed lines of the file:
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@@
 </autorouter>
 <elements>
-<element name="D1" library="diode-tvs" package="SMC" value="SMCJ36CA" x="50.720625" y="21.669375" smashed="yes" rot="R270">
+<element name="D1" library="kaktus" package="SMC" value="SMCJ36CA" x="50.720625" y="21.669375" smashed="yes" rot="R270">
 <attribute name="NAME" x="47.18225" y="25.663375" size="0.8128" layer="25" font="vector"/>
 <attribute name="VALUE" x="46.091625" y="25.128375" size="1.27" layer="27" rot="R270"/>
@@
 <attribute name="VALUE" x="9.293225" y="10.43305" size="2.0828" layer="27" ratio="10" rot="SR270"/>
 </element>
-<element name="D6" library="diode" package="DO-214AC" value="SMAJ45CA" x="44.45" y="38.496875" smashed="yes" rot="R270">
+<element name="D6" library="kaktus" package="DO-214AC" value="SMAJ45CA" x="44.45" y="38.496875" smashed="yes" rot="R270">
 <attribute name="NAME" x="43.65625" y="41.513125" size="0.8128" layer="25" font="vector"/>
 <attribute name="VALUE" x="41.275" y="41.036875" size="1.27" layer="27" rot="R270"/>
 </element>
-<element name="D7" library="diode" package="DO-214AC" value="SMAJ45CA" x="48.26" y="38.496875" smashed="yes" rot="R270">
+<element name="D7" library="kaktus" package="DO-214AC" value="SMAJ45CA" x="48.26" y="38.496875" smashed="yes" rot="R270">
 <attribute name="NAME" x="47.9425" y="41.513125" size="0.8128" layer="25" font="vector"/>
 <attribute name="VALUE" x="45.085" y="41.036875" size="1.27" layer="27" rot="R270"/>
@@
 <attribute name="VALUE" x="7.77875" y="42.545" size="1.27" layer="27" rot="R180"/>
 </element>
-<element name="D8" library="diode" package="DO-214AC" value="SMAJ12CA" x="48.26" y="30.48" smashed="yes" rot="R270">
+<element name="D8" library="kaktus" package="DO-214AC" value="SMAJ12CA" x="48.26" y="30.48" smashed="yes" rot="R270">
 <attribute name="NAME" x="50.00625" y="31.353125" size="0.8128" layer="25" font="vector"/>
 <attribute name="VALUE" x="45.085" y="33.02" size="1.27" layer="27" rot="R270"/>
