File: Schematic-and-BOM/MightyWatt R3.brd (EAGLE design)
At the start: 64.8 x 53.3 mm, 93 parts, among them IC1 TLV271IDBVR, IC2 MAX4619EUE, IC3 OPA365AIDBVR, IC4 TS5A3166, IC5 INA225, IC6 ADS1115IDGST, IC7 TLV2372IDGK, IC8 AD5691RAD5691R, IC9 LM2766M6, T1 IXTH75N10L2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

Commit message: Rearranged wires to prevent solder bridges
Routing:
- net CCCV: track 83.3 -> 86.6 mm
- net N$10: track 16.1 -> 17.3 mm
- net GND: track 85.4 -> 86.4 mm
- net VCCIO: track 245.3 -> 246.1 mm
- net IGAIN: track 67.2 -> 67.8 mm
Other:
- board text added: "kaktus circuits Czech Republic 2020 CC-BY-SA jpolonsky@gmail.com"
- board text removed: "kaktus circuits Czech Republic 2017 CC-BY-SA jpolonsky@gmail.com"
